File: KiCad/AYOM - Power Supply Front Panel.kicad_pcb (KiCad board)
At the start: 2 copper layers, 3 parts

Commit message: Updated Gerbers and archive
Parts:
- added svg2mod: G***, Custom_Graphics:PS_Panel_Copper_Mask, F.Cu at (108.1, 38.6)
- added svg2mod: G***, Custom_Graphics:PS_Panel_Copper, F.Cu at (108.1, 38.6)
- added svg2mod: G***, Custom_Graphics:PS_Panel_Silkscreen, F.Cu at (108.1, 38.6)
- added svg2mod: G***, Custom_Graphics:PS_Panel_EdgeCuts, F.Cu at (108.1, 38.6)
Routing:
- added copper zone on B.Cu, net (none)
- added copper zone on F.Cu, net (none)
Other:
- board outline added: 40.3 x 128.5 mm
